File: Design_final/Design_final.brd (EAGLE design)
At the start: 69.5 x 73.7 mm, 34 parts, among them IC1 LF353D, IC2 7815T, IC3 7805L, IC4 MCP601P

Commit message: New final
Routing:
- net N$13: track 40.1 -> 10.1 mm
- net N$7: track 28.5 -> 5.72 mm
- net V+: track 116.7 -> 128.4 mm
- net N$6: track 32.7 -> 41.1 mm
- net +5V: track 59.0 -> 65.3 mm
- net N$9: track 35.7 -> 41.1 mm
- net +3V3: track 32.9 -> 36.9 mm
- net N$4: track 47.3 -> 50.5 mm
- net N$15: track 19.9 -> 22.3 mm
- net N$8: track 8.33 -> 9.81 mm
- net N$2: track 52.9 -> 51.5 mm
- net N$3: track 5.24 -> 4.17 mm
- net N$1: track 43.2 -> 43.8 mm
